File: FPGA_GPIO.kicad_sch (KiCad schematic)
At the start: 3 parts, among them J1 DF12NC_3.0_-60DS-0.5V_51_, J2 DF12NC_3.0_-60DS-0.5V_51_, U4 LFMXO5-25

Commit message: relay unit
Parts:
- removed J1, J2: DF12NC_3.0_-60DS-0.5V_51_, DF12NC_3.0_60DS-0.5V:HRS_DF12NC_3.0_-60DS-0.5V_51_, symbol DF12NC_3.0_-60DS-0.5V_51_:DF12NC_3.0_-60DS-0.5V_51_
- added J1, J3: Conn_02x10_Top_Bottom, Connector_PinHeader_1.27mm:PinHeader_2x10_P1.27mm_Vertical_SMD, symbol Connector_Generic:Conn_02x10_Top_Bottom
- added J13: Conn_01x08_Pin, Connector_PinHeader_1.27mm:PinHeader_1x08_P1.27mm_Vertical, symbol Connector:Conn_01x08_Pin
- added R184, R185: 1k, Resistor_SMD:R_0402_1005Metric, symbol Device:R
- added R186, R187, R188, R189: 4.7k, Resistor_SMD:R_0402_1005Metric, symbol Device:R
- added unit 13 of U4
Connections:
- net +3V3_BANK: now also J13.1 (Pin_1), R184.1, R185.1, R186.1, R187.1, R188.1
- net GND: now also J13.7 (Pin_7), R189.2
- net PWM0: now also J3.9 (Pin_9)
- net PWM1: now also J3.10 (Pin_10)
- net PWM2: now also J3.7 (Pin_7)
- net PWM3: now also J3.8 (Pin_8)
- net PWM30: now also J1.11 (Pin_11)
- net PWM31: now also J1.12 (Pin_12)
- net PWM32: now also J1.13 (Pin_13)
- net PWM33: now also J1.14 (Pin_14)
- net PWM34: now also J1.15 (Pin_15)
- net PWM35: now also J1.16 (Pin_16)
- net PWM36: now also J1.17 (Pin_17)
- net PWM37: now also J1.18 (Pin_18)
- net PWM38: now also J1.19 (Pin_19)
- net PWM39: now also J1.20 (Pin_20)
- net PWM4: now also J3.5 (Pin_5)
- net PWM5: now also J3.6 (Pin_6)
- net PWM6: now also J3.3 (Pin_3)
- net PWM7: now also J3.4 (Pin_4)
- net PWM8: now also J3.1 (Pin_1)
- net PWM9: now also J3.2 (Pin_2)
- net dim_sw0_N: now also J3.13 (Pin_13)
- net dim_sw0_P: now also J3.11 (Pin_11)
- net dim_sw1_N: now also J3.14 (Pin_14)
- net dim_sw1_P: now also J3.12 (Pin_12)
- net dim_sw2_N: now also J3.17 (Pin_17)
- net dim_sw2_P: now also J3.15 (Pin_15)
- net dim_sw3_N: now also J3.18 (Pin_18)
- net dim_sw3_P: now also J3.16 (Pin_16)
- net dim_sw4_N: now also J3.20 (Pin_20)
- net dim_sw4_P: now also J3.19 (Pin_19)
- net dim_sw5_N: now also J1.2 (Pin_2)
- net dim_sw5_P: now also J1.1 (Pin_1)
- net dim_sw6_N: now also J1.3 (Pin_3)
- net dim_sw6_P: now also J1.5 (Pin_5)
- net dim_sw7_N: now also J1.4 (Pin_4)
- net dim_sw7_P: now also J1.6 (Pin_6)
- net dim_sw8_N: now also J1.7 (Pin_7)
- net dim_sw8_P: now also J1.9 (Pin_9)
- net dim_sw9_N: now also J1.8 (Pin_8)
- net dim_sw9_P: now also J1.10 (Pin_10)
- new net DONE: U4.A11 (INITN)
- new net INIT: U4.A13 (DONE)
- new net JTAG_EN: J13.5 (Pin_5), R184.2, U4.B16 (JTAG_EN)
- new net NX_TCK: J13.8 (Pin_8), R189.1, U4.G10 (TCK/SCLK/PMU_EXT_CLK)
- new net NX_TDI: J13.3 (Pin_3), R187.2, U4.F16 (TDI/SSI/SD0/S5_OUT)
- new net NX_TDO: J13.2 (Pin_2), R188.2, U4.F10 (TDO/SSO/SD1/S3_OUT)
- new net NX_TMS: J13.6 (Pin_6), R186.2, U4.E14 (TMS/SCSN/S5_IN)
- new net PROGRAMN: R185.2, U4.A12 (PROGRAMN)
- no-connect marks 0 -> 1
Other:
- added sheet PWM (PWM.kicad_sch)
- moved on the sheet: U4K
