File: FPGA_machX05.kicad_sch (KiCad schematic)
At the start: 0 parts

Commit message: relay unit
Other:
- removed sheet FTDI
- added sheet sw (dim_sw.kicad_sch)
Changed lines of the file:
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@@
 	(paper "A4")
 	(sheet
-		(at 99.822 26.67)
-		(size 12.7 3.81)
+		(at 120.65 38.1)
+		(size 34.29 8.89)
 		(fields_autoplaced yes)
 		(stroke
@@
 			(color 0 0 0 0.0000)
 		)
-		(property "Sheetname" "FTDI"
-			(at 99.822 25.9584 0)
+		(property "Sheetname" "sw"
+			(at 120.65 37.3884 0)
 			(effects
 				(font
@@
 			)
 		)
-		(property "Sheetfile" "FTDI.kicad_sch"
-			(at 99.822 31.0646 0)
+		(property "Sheetfile" "dim_sw.kicad_sch"
+			(at 120.65 47.5746 0)
 			(effects
 				(font
@@
 			(project "home_auto"
 				(path "/68de2dd7-8f08-479b-94c5-c7847794fd33/0646acc6-79c1-4e67-b684-df663024146f"
-					(page "7")
+					(page "79")
 				)
 			)
@@
 	)
 	(sheet
-		(at 42.164 26.67)
-		(size 12.7 3.81)
+		(at 29.21 38.1)
+		(size 29.21 8.89)
 		(fields_autoplaced yes)
 		(stroke
@@
 		)
 		(property "Sheetname" "POWER"
-			(at 42.164 25.9584 0)
+			(at 29.21 37.3884 0)
 			(effects
 				(font
@@
 		)
 		(property "Sheetfile" "POWER.kicad_sch"
-			(at 42.164 31.0646 0)
+			(at 29.21 47.5746 0)
 			(effects
 				(font
@@
 	)
 	(sheet
-		(at 71.12 26.67)
-		(size 12.7 3.81)
+		(at 36.83 67.056)
+		(size 43.688 13.462)
 		(fields_autoplaced yes)
 		(stroke
@@
 		)
 		(property "Sheetname" "FPGA_GPIO"
-			(at 71.12 25.9584 0)
+			(at 36.83 66.3444 0)
 			(effects
 				(font
@@
 		)
 		(property "Sheetfile" "FPGA_GPIO.kicad_sch"
-			(at 71.12 31.0646 0)
+			(at 36.83 81.1026 0)
 			(effects
 				(font
